File: shield/JVS-IO/JVS-IO.kicad_sch (KiCad schematic)
At the start: 47 parts, among them J1 Conn_01x08, J2 Conn_01x03, J3 Conn_01x03, J4 Conn_01x03, K1 G6S-2, Q1 BC847, Q2 BC847, Q3 BC847, Q4 BC847, U1 MAX485E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

Commit message: Fixed errant bugs
Parts:
- R13, R14: value 103 -> 102
Changed lines of the file:
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@@
     (in_bom yes) (on_board yes)
     (property "Reference" "R13" (id 0) (at 92.075 140.335 90))
-    (property "Value" "103" (id 1) (at 92.71 142.24 90))
+    (property "Value" "102" (id 1) (at 92.71 142.24 90))
     (property "Footprint" "Resistor_SMD:R_1206_3216Metric" (id 2) (at 92.71 144.78 0)
       (effects (font (size 1.27 1.27)) hide)
@@
     (in_bom yes) (on_board yes)
     (property "Reference" "R14" (id 0) (at 95.25 154.305 90))
-    (property "Value" "103" (id 1) (at 95.885 156.21 90))
+    (property "Value" "102" (id 1) (at 95.885 156.21 90))
     (property "Footprint" "Resistor_SMD:R_1206_3216Metric" (id 2) (at 95.885 158.75 0)
       (effects (font (size 1.27 1.27)) hide)
@@
     )
     (path "/3236e942-6e02-4559-a957-ea58a9f439fc"
-      (reference "R13") (unit 1) (value "103") (footprint "Resistor_SMD:R_1206_3216Metric")
+      (reference "R13") (unit 1) (value "102") (footprint "Resistor_SMD:R_1206_3216Metric")
     )
     (path "/b241b830-f726-45f1-8a7b-e737c306a76b"
-      (reference "R14") (unit 1) (value "103") (footprint "Resistor_SMD:R_1206_3216Metric")
+      (reference "R14") (unit 1) (value "102") (footprint "Resistor_SMD:R_1206_3216Metric")
     )
     (path "/e4331afd-0e42-468d-934f-3b5b019cd145"
